File: sensors/_uart.kicad_sch (KiCad schematic)
At the start: 19 parts, among them J5 JP_GPS, J6 JP_RADIO, U1 SC16IS752IPW

Commit message: use 2x8 for ADC header; added part numbers
Parts:
- J5, J6: Part (none) -> HCZZ0001-6
- R6, R9: Part C25744 -> FRC0402F4700TS
- U1: Part (none) -> SC16IS752IPW,128
Changed lines of the file:
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@@
 			)
 		)
-		(property "Part" "C25744"
+		(property "Part" "FRC0402F4700TS"
 			(at 271.78 81.28 0)
 			(hide yes)
@@
 			)
 		)
-		(property "Part" ""
+		(property "Part" "HCZZ0001-6"
 			(at 43.18 212.09 0)
 			(hide yes)
@@
 			)
 		)
-		(property "Part" "C25744"
+		(property "Part" "FRC0402F4700TS"
 			(at 327.66 81.28 0)
 			(hide yes)
@@
 			)
 		)
+		(property "Part" "SC16IS752IPW,128"
+			(at 152.4 99.06 0)
+			(hide yes)
+			(show_name no)
+			(do_not_autoplace no)
+			(effects
+				(font
+					(size 1.27 1.27)
+				)
+			)
+		)
 		(pin "12"
 		)
@@
 			)
 		)
-		(property "Part" ""
+		(property "Part" "HCZZ0001-6"
 			(at 43.18 242.57 0)
 			(hide yes)
