File: sensors/_imu.kicad_sch (KiCad schematic)
At the start: 4 parts, among them U3 ICM-42605

Commit message: add Vref
Other:
- title: (none) -> PilotPi: Sensors
Changed lines of the file:
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@@
 	(generator_version "10.0")
 	(paper "A4")
+	(title_block
+		(title "PilotPi: Sensors")
+		(date "15 nov 2012")
+		(rev "4")
+	)
 	(junction
 		(at 152.4 74.93)

Commit message: added JP_VOLTS, Vref select jumper; VBAT_ADC Jumper
Parts:
- C6: Part (none) -> CC0402X7R50V104KN
Changed lines of the file:
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@@
 			)
 		)
-		(property "Part" ""
+		(property "Part" "CC0402X7R50V104KN"
 			(at 228.6 97.79 0)
 			(hide yes)

Commit message: use CLK out from CAN controller for UART (use 16 MHz instead of 14.7456MHz); minor changes
Parts:
- C6: value 100nF (104) 10% 16V -> 100nF 10% 16V
- C7: value 220nF (224) 10% 16V -> 220nF 10% 16V
- C8: value 10nF (103) 10% 50V -> 10nF 10% 50V
Changed lines of the file:
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@@
 			)
 		)
-		(property "Value" "100nF (104) 10% 16V"
+		(property "Value" "100nF 10% 16V"
 			(at 223.266 106.172 90)
 			(show_name no)
@@
 			)
 		)
-		(property "Value" "220nF (224) 10% 16V"
+		(property "Value" "220nF 10% 16V"
 			(at 234.696 106.172 90)
 			(show_name no)
@@
 			)
 		)
-		(property "Value" "10nF (103) 10% 50V"
+		(property "Value" "10nF 10% 50V"
 			(at 246.126 106.172 90)
 			(show_name no)

Commit message: use 2x8 for ADC header; added part numbers
Parts:
- C7: Part (none) -> TCC0402X7R224K250ATM
- C8: Part (none) -> FN15X103J500PNG
- U3: Part (none) -> ICM-42605-HXY
Changed lines of the file:
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@@
 			)
 		)
-		(property "Part" ""
+		(property "Part" "TCC0402X7R224K250ATM"
 			(at 240.03 97.79 0)
 			(hide yes)
@@
 			)
 		)
-		(property "Part" ""
+		(property "Part" "FN15X103J500PNG"
 			(at 251.46 97.79 0)
 			(hide yes)
@@
 			)
 		)
-		(property "Part" ""
+		(property "Part" "ICM-42605-HXY"
 			(at 154.94 97.79 0)
 			(hide yes)

Commit message: replace MS561101 pressure sensor with SPL06-001
Parts:
- C6: Part CC0402X7R50V104KN -> CL05B104KB54PNC
- C7: Part TCC0402X7R224K250ATM -> CL05B224KO5NNNC
- C8: Part FN15X103J500PNG -> CL05B103KB5NNNC
Changed lines of the file:
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@@
 			)
 		)
-		(property "Part" "CC0402X7R50V104KN"
+		(property "Part" "CL05B104KB54PNC"
 			(at 228.6 97.79 0)
 			(hide yes)
@@
 			)
 		)
-		(property "Part" "TCC0402X7R224K250ATM"
+		(property "Part" "CL05B224KO5NNNC"
 			(at 240.03 97.79 0)
 			(hide yes)
@@
 			)
 		)
-		(property "Part" "FN15X103J500PNG"
+		(property "Part" "CL05B103KB5NNNC"
 			(at 251.46 97.79 0)
 			(hide yes)

Commit message: use series resistor for external clk; add 1uF caps
Parts:
- added C23: 1uF (105) 10% 50V, Capacitor_SMD:C_0603_1608Metric, symbol Device:C
Connections:
- net +3V3: now also C23.1
- net GND: now also C23.2
