File: sensors/_mag.kicad_sch (KiCad schematic)
At the start: 3 parts, among them U4 IST8310

Commit message: add Vref
Other:
- title: (none) -> PilotPi: Sensors
Changed lines of the file:
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@@
 	(generator_version "10.0")
 	(paper "A4")
+	(title_block
+		(title "PilotPi: Sensors")
+		(date "15 nov 2012")
+		(rev "4")
+	)
 	(junction
 		(at 146.05 76.2)

Commit message: added JP_VOLTS, Vref select jumper; VBAT_ADC Jumper
Parts:
- C9: Part (none) -> CC0402X7R50V104KN
Changed lines of the file:
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@@
 			)
 		)
-		(property "Part" ""
+		(property "Part" "CC0402X7R50V104KN"
 			(at 199.39 92.71 0)
 			(hide yes)

Commit message: use CLK out from CAN controller for UART (use 16 MHz instead of 14.7456MHz); minor changes
Parts:
- C10: value 470nF (474) 10% 25V -> 470nF 10% 25V
- C9: value 100nF (104) 10% 16V -> 100nF 10% 16V
Changed lines of the file:
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@@
 			)
 		)
-		(property "Value" "470nF (474) 10% 25V"
+		(property "Value" "470nF 10% 25V"
 			(at 162.052 107.95 0)
 			(show_name no)
@@
 			)
 		)
-		(property "Value" "100nF (104) 10% 16V"
+		(property "Value" "100nF 10% 16V"
 			(at 194.056 101.092 90)
 			(show_name no)

Commit message: use 2x8 for ADC header; added part numbers
Parts:
- C10: Part (none) -> TCC0402X5R474K250AT
Changed lines of the file:
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@@
 			)
 		)
-		(property "Part" ""
+		(property "Part" "TCC0402X5R474K250AT"
 			(at 158.75 106.68 0)
 			(hide yes)

Commit message: replace MS561101 pressure sensor with SPL06-001
Parts:
- C10: Part TCC0402X5R474K250AT -> CL10B474KA8NNNC
- C9: Part CC0402X7R50V104KN -> CL05B104KB54PNC
Changed lines of the file:
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@@
 			)
 		)
-		(property "Part" "TCC0402X5R474K250AT"
+		(property "Part" "CL10B474KA8NNNC"
 			(at 158.75 106.68 0)
 			(hide yes)
@@
 			)
 		)
-		(property "Part" "CC0402X7R50V104KN"
+		(property "Part" "CL05B104KB54PNC"
 			(at 199.39 92.71 0)
 			(hide yes)

Commit message: use series resistor for external clk; add 1uF caps
Parts:
- added C24: 1uF (105) 10% 50V, Capacitor_SMD:C_0603_1608Metric, symbol Device:C
Connections:
- net +3V3: now also C24.1
- net GND: now also C24.2
