File: sensors/_dshot.kicad_sch (KiCad schematic)
At the start: 10 parts, among them U10 74HCT595

Commit message: lots of changes
Parts:
- U10: value 74HCT595 -> 74AHCT595; footprint Package_SO:SOP-16_4.4x10.4mm_P1.27mm -> pilotpi:WQFN-16-1EP_2.5x3.5mm_P0.5mm; Part HX74HC595-S -> SN74AHCT595BQBR
Changed lines of the file:
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@@
 			)
 		)
-		(property "Value" "74HCT595"
+		(property "Value" "74AHCT595"
 			(at 144.3833 85.09 0)
 			(show_name no)
@@
 			)
 		)
-		(property "Footprint" "Package_SO:SOP-16_4.4x10.4mm_P1.27mm"
+		(property "Footprint" "pilotpi:WQFN-16-1EP_2.5x3.5mm_P0.5mm"
 			(at 142.24 100.33 0)
 			(hide yes)
@@
 			)
 		)
-		(property "Part" "HX74HC595-S"
+		(property "Part" "SN74AHCT595BQBR"
 			(at 142.24 100.33 0)
 			(hide yes)

Commit message: replace MS561101 pressure sensor with SPL06-001
Parts:
- C18: Part CC0402X7R50V104KN -> CL05B104KB54PNC
- R38, R39, R40, R41, R42, R43, R44, R45: Part RC0402FR-0722RL -> 0402WGF220JTCE
Changed lines of the file:
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@@
 			)
 		)
-		(property "Part" "RC0402FR-0722RL"
+		(property "Part" "0402WGF220JTCE"
 			(at 180.34 105.41 0)
 			(hide yes)
@@
 			)
 		)
-		(property "Part" "RC0402FR-0722RL"
+		(property "Part" "0402WGF220JTCE"
 			(at 190.5 107.95 0)
 			(hide yes)
@@
 			)
 		)
-		(property "Part" "RC0402FR-0722RL"
+		(property "Part" "0402WGF220JTCE"
 			(at 160.02 100.33 0)
 			(hide yes)
@@
 			)
 		)
-		(property "Part" "RC0402FR-0722RL"
+		(property "Part" "0402WGF220JTCE"
 			(at 180.34 95.25 0)
 			(hide yes)
@@
 			)
 		)
-		(property "Part" "RC0402FR-0722RL"
+		(property "Part" "0402WGF220JTCE"
 			(at 170.18 102.87 0)
 			(hide yes)
@@
 			)
 		)
-		(property "Part" "CC0402X7R50V104KN"
+		(property "Part" "CL05B104KB54PNC"
 			(at 82.55 101.6 0)
 			(hide yes)
@@
 			)
 		)
-		(property "Part" "RC0402FR-0722RL"
+		(property "Part" "0402WGF220JTCE"
 			(at 170.18 92.71 0)
 			(hide yes)
@@
 			)
 		)
-		(property "Part" "RC0402FR-0722RL"
+		(property "Part" "0402WGF220JTCE"
 			(at 190.5 97.79 0)
 			(hide yes)
@@
 			)
 		)
-		(property "Part" "RC0402FR-0722RL"
+		(property "Part" "0402WGF220JTCE"
 			(at 160.02 90.17 0)
 			(hide yes)
