File: sensors/_pressure.kicad_sch (KiCad schematic)
At the start: 3 parts, among them U5 SPL06-001

Commit message: replace barometer; exclude solder jumpers from bom/pos
Parts:
- U5: value SPL06-001 -> SPA06-003; Part SPL06-001 -> SPA06-003
Changed lines of the file:
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@@
 			)
 		)
-		(property "Value" "SPL06-001"
+		(property "Value" "SPA06-003"
 			(at 149.86 91.4399 0)
 			(show_name no)
@@
 			)
 		)
-		(property "Datasheet" "https://www.te.com/commerce/DocumentDelivery/DDEController?Action=showdoc&DocId=Data+Sheet%7FMS5607-02BA03%7FB2%7Fpdf%7FEnglish%7FENG_DS_MS5607-02BA03_B2.pdf%7FCAT-BLPS0035"
+		(property "Datasheet" "https://jlcpcb.com/api/file/downloadByFileSystemAccessId/8604442257579782144"
 			(at 140.97 90.17 0)
 			(hide yes)
@@
 			)
 		)
-		(property "Description" "Barometric pressure sensor, 20cm resolution, 10 to 1200 mbar, I2C and SPI interface up to 20MHz, LGA-8"
+		(property "Description" "-40℃~+85℃ 0.95mm 1.7V~3.6V 1.7uA 2.5mm 2mm SPI、I2C LGA-8(2x2.5) Pressure Sensors ROHS"
 			(at 140.97 90.17 0)
 			(hide yes)
@@
 			)
 		)
-		(property "Part" "SPL06-001"
+		(property "Part" "SPA06-003"
 			(at 140.97 90.17 0)
 			(hide yes)
