File: sensors/_rs485.kicad_sch (KiCad schematic)
At the start: 5 parts, among them U11 SP3485EN

Commit message: series resistor to protect RO
Parts:
- added R47: 150Ω ±1%, Resistor_SMD:R_0402_1005Metric, symbol Device:R
Connections:
- net RO: now also R47.1; no longer U11.1 (RO)
- new net: R47.2, U11.1 (RO)
Changed lines of the file:
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@@
 	(wire
 		(pts
-			(xy 124.46 83.82) (xy 139.7 83.82)
+			(xy 134.62 83.82) (xy 139.7 83.82)
 		)
 		(stroke
@@
 		(pts
 			(xy 189.23 95.25) (xy 199.39 95.25)
+		)
+		(stroke
+			(width 0)
+			(type default)
+		)
+	)
+	(wire
+		(pts
+			(xy 124.46 83.82) (xy 127 83.82)
 		)
 		(stroke
@@
 					(unit 1)
 				)
+			)
+		)
+	)
+	(symbol
+		(lib_id "Device:R")
+		(at 130.81 83.82 90)
+		(unit 1)
+		(body_style 1)
+		(exclude_from_sim no)
+		(in_bom yes)
+		(on_board yes)
+		(in_pos_files yes)
+		(dnp no)
+		(fields_autoplaced yes)
+		(property "Reference" "R47"
+			(at 130.81 77.47 90)
+			(show_name no)
+			(do_not_autoplace no)
+			(effects
+				(font
+					(size 1.27 1.27)
+				)
+			)
+		)
+		(property "Value" "150Ω ±1%"
+			(at 130.81 80.01 90)
+			(show_name no)
+			(do_not_autoplace no)
+			(effects
+				(font
+					(size 1.27 1.27)
+				)
+			)
+		)
+		(property "Footprint" "Resistor_SMD:R_0402_1005Metric"
+			(at 130.81 85.598 90)
+			(hide yes)
+			(show_name no)
+			(do_not_autoplace no)
+			(effects
+				(font
+					(size 1.27 1.27)
+				)
+			)
+		)
+		(property "Datasheet" ""
+			(at 130.81 83.82 0)
+			(hide yes)
+			(show_name no)
+			(do_not_autoplace no)
+			(effects
+				(font
+					(size 1.27 1.27)
+				)
+			)
+		)
+		(property "Description" "Resistor"
+			(at 130.81 83.82 0)
+			(hide yes)
+			(show_name no)
+			(do_not_autoplace no)
+			(effects
+				(font
+					(size 1.27 1.27)
+				)
+			)
+		)
+		(property "Part" ""
+			(at 130.81 83.82 0)
+			(hide yes)
+			(show_name no)
+			(do_not_autoplace no)
+			(effects
+				(font
+					(size 1.27 1.27)
+				)
+			)
+		)
+		(pin "2"
+		)
+		(pin "1"
+		)
+		(instances
+			(project "sensors"
+				(path "/e63e39d7-6ac0-4ffd-8aa3-1841a4541b55/1f34d345-dfef-4499-b9fc-3fc6a0420831"
+					(reference "R47")
+					(unit 1)
+				)

Commit message: use series resistor for external clk; add 1uF caps
Parts:
- added C29: 1uF (105) 10% 50V, Capacitor_SMD:C_0603_1608Metric, symbol Device:C
Connections:
- net +3V3: now also C29.1
- net GND: now also C29.2
Other:
- moved on the sheet: C21

Commit message: add missing part numbers
Parts:
- D6: Part (none) -> PSM712-LF-T7
- R46: Part (none) -> 0402WGF1200TCE
- R47: footprint Resistor_SMD:R_0402_1005Metric -> Resistor_SMD:R_0603_1608Metric; Part (none) -> 0603WAF1500T5E
- U11: Part (none) -> SP3485EN-L/TR
Changed lines of the file:
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@@
+			)
+		)
+		(property "Part" "SP3485EN-L/TR"
+			(at 149.86 88.9 0)
+			(hide yes)
+			(show_name no)
+			(do_not_autoplace no)
+			(effects
+				(font
+					(size 1.27 1.27)
+				)
 			)
 		)
@@
 			)
 		)
-		(property "Footprint" "Resistor_SMD:R_0402_1005Metric"
+		(property "Footprint" "Resistor_SMD:R_0603_1608Metric"
 			(at 130.81 85.598 90)
 			(hide yes)
@@
 			)
 		)
-		(property "Part" ""
+		(property "Part" "0603WAF1500T5E"
 			(at 130.81 83.82 0)
 			(hide yes)
@@
 			)
 		)
-		(property "Part" ""
+		(property "Part" "0402WGF1200TCE"
 			(at 199.39 78.74 0)
 			(hide yes)
@@
 			(hide yes)
 			(show_name no)
+			(do_not_autoplace no)
+			(effects
+				(font
+					(size 1.27 1.27)
+				)
+			)
+		)
+		(property "Part" "PSM712-LF-T7"
+			(at 189.23 83.82 90)
+			(hide yes)
+			(show_name no)

Commit message: remove old part no's
Parts:
- JP5: Part 2541WV-2X01P -> (none)
Changed lines of the file:
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@@
 			)
 		)
-		(property "Part" "2541WV-2X01P"
+		(property "Part" ""
 			(at 199.39 88.9 0)
 			(hide yes)

Commit message: replace barometer; exclude solder jumpers from bom/pos
Parts:
- JP5: now left out of the parts list
Changed lines of the file:
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@@
 		(body_style 1)
 		(exclude_from_sim no)
-		(in_bom yes)
+		(in_bom no)
 		(on_board yes)
-		(in_pos_files yes)
+		(in_pos_files no)
 		(dnp no)
 		(fields_autoplaced yes)
