File: sensors/_boot_mode.kicad_sch (KiCad schematic)
At the start: 2 parts, among them SW2 SW_SPDT_321

Commit message: add Vref
Other:
- title: (none) -> PilotPi: Sensors
Changed lines of the file:
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@@
 	(generator_version "10.0")
 	(paper "A4")
+	(title_block
+		(title "PilotPi: Sensors")
+		(date "15 nov 2012")
+		(rev "4")
+	)
 	(text "ON"
 		(exclude_from_sim no)

Commit message: use CLK out from CAN controller for UART (use 16 MHz instead of 14.7456MHz); minor changes
Parts:
- R35: value 10KΩ (1002) ±1% -> 10KΩ ±1%
Changed lines of the file:
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@@
 			)
 		)
-		(property "Value" "10KΩ (1002) ±1%"
+		(property "Value" "10KΩ ±1%"
 			(at 125.984 95.25 90)
 			(show_name no)

Commit message: use 2x8 for ADC header; added part numbers
Parts:
- R35: Part (none) -> C25744
Changed lines of the file:
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@@
 			)
 		)
-		(property "Part" ""
+		(property "Part" "C25744"
 			(at 132.08 92.71 0)
 			(hide yes)

Commit message: fix 5V on GPIO
Connections:
- net +5V renamed +3V3
Changed lines of the file:
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@@
-	)
-	(symbol
-		(lib_id "power:+5V")
-		(at 124.46 88.9 0)
-		(unit 1)
-		(body_style 1)
-		(exclude_from_sim no)
-		(in_bom yes)
-		(on_board yes)
-		(in_pos_files yes)
-		(dnp no)
-		(property "Reference" "#PWR072"
-			(at 124.46 92.71 0)
-			(hide yes)
-			(show_name no)
-			(do_not_autoplace no)
-			(effects
-				(font
-					(size 1.27 1.27)
-				)
-			)
-		)
-		(property "Value" "+5V"
-			(at 124.8283 84.5756 0)
-			(show_name no)
-			(do_not_autoplace no)
-			(effects
-				(font
-					(size 1.27 1.27)
-				)
-			)
-		)
-		(property "Footprint" ""
-			(at 124.46 88.9 0)
-			(show_name no)
-			(do_not_autoplace no)
-			(effects
-				(font
-					(size 1.27 1.27)
-				)
-			)
-		)
-		(property "Datasheet" ""
-			(at 124.46 88.9 0)
-			(show_name no)
-			(do_not_autoplace no)
-			(effects
-				(font
-					(size 1.27 1.27)
-				)
-			)
-		)
-		(property "Description" "Power symbol creates a global label with name \"+5V\""
-			(at 124.46 88.9 0)
-			(hide yes)
-			(show_name no)
-			(do_not_autoplace no)
-			(effects
-				(font
-					(size 1.27 1.27)
-				)
-			)
-		)
-		(pin "1"
-		)
-		(instances
-			(project "sensors"
-				(path "/e63e39d7-6ac0-4ffd-8aa3-1841a4541b55/6d51b619-4bc5-4344-81ae-260f6b2b0bff"
-					(reference "#PWR072")
-					(unit 1)
-				)
-			)
-		)
 	)
 	(symbol
@@
 					(unit 1)
 				)
+			)
+		)
+	)
+	(symbol
+		(lib_id "power:+3.3V")
+		(at 124.46 88.9 0)
+		(unit 1)
+		(body_style 1)
+		(exclude_from_sim no)
+		(in_bom yes)
+		(on_board yes)
+		(in_pos_files yes)
+		(dnp no)
+		(property "Reference" "#PWR084"
+			(at 124.46 92.71 0)
+			(hide yes)
+			(show_name no)
+			(do_not_autoplace no)
+			(effects
+				(font
+					(size 1.27 1.27)
+				)
+			)
+		)
+		(property "Value" "+3V3"
+			(at 124.8283 84.5756 0)
+			(show_name no)
+			(do_not_autoplace no)
+			(effects
+				(font
+					(size 1.27 1.27)
+				)
+			)
+		)
+		(property "Footprint" ""
+			(at 124.46 88.9 0)
+			(show_name no)
+			(do_not_autoplace no)
+			(effects
+				(font
+					(size 1.27 1.27)
+				)
+			)
+		)
+		(property "Datasheet" ""
+			(at 124.46 88.9 0)
+			(show_name no)
+			(do_not_autoplace no)
+			(effects
+				(font
+					(size 1.27 1.27)
+				)
+			)
+		)
+		(property "Description" "Power symbol creates a global label with name \"+3.3V\""
+			(at 124.46 88.9 0)
+			(hide yes)
+			(show_name no)
+			(do_not_autoplace no)
+			(effects
+				(font
+					(size 1.27 1.27)
+				)
+			)
+		)
+		(pin "1"
+		)
+		(instances
+			(project "sensors"
+				(path "/e63e39d7-6ac0-4ffd-8aa3-1841a4541b55/6d51b619-4bc5-4344-81ae-260f6b2b0bff"
+					(reference "#PWR084")
+					(unit 1)
+				)
