File: sensors/_pwm.kicad_sch (KiCad schematic)
At the start: 22 parts, among them U2 PCA9685PW, Y2 25M-3225

Commit message: use 3V3 to power PCA9685
Connections:
- net +5V is gone; now on net +3V3: C20.1, C4.1, U2.28 (VDD)
