File: power/_xl4015.kicad_sch (KiCad schematic)
At the start: 11 parts, among them U1 XL4015

Commit message: lots of changes
Parts:
- C1: Part (none) -> VT1H221M1010
- C2, C3, C4: Part (none) -> 0805B105M500AT
- C5: Part (none) -> TCC0805X7R333K500DTS
- C6: Part (none) -> RVT1C471M0810
- D1: Part (none) -> SS54
- R1: Part (none) -> RCA0510KFLF
- R2: Part (none) -> SCR0805F3K3
Changed lines of the file:
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@@
 		(date "15 nov 2012")
 		(rev "4")
+		(comment 1 "VCC -> 5V switching PSU")
 	)
 	(junction
@@
 			)
 		)
+		(property "Part" "RVT1C471M0810"
+			(at 262.89 148.59 0)
+			(hide yes)
+			(show_name no)
+			(do_not_autoplace no)
+			(effects
+				(font
+					(size 1.27 1.27)
+				)
+			)
+		)
 		(pin "1"
 		)
@@
 			)
 		)
+		(property "Part" "0805B105M500AT"
+			(at 142.24 146.05 0)
+			(hide yes)
+			(show_name no)
+			(do_not_autoplace no)
+			(effects
+				(font
+					(size 1.27 1.27)
+				)
+			)
+		)
 		(pin "1"
 		)
@@
 			)
 		)
+		(property "Part" "VT1H221M1010"
+			(at 121.92 146.05 0)
+			(hide yes)
+			(show_name no)
+			(do_not_autoplace no)
+			(effects
+				(font
+					(size 1.27 1.27)
+				)
+			)
+		)
 		(pin "1"
 		)
@@
 			)
 		)
+		(property "Part" "0805B105M500AT"
+			(at 166.37 135.89 0)
+			(hide yes)
+			(show_name no)
+			(do_not_autoplace no)
+			(effects
+				(font
+					(size 1.27 1.27)
+				)
+			)
+		)
 		(pin "1"
 		)
@@
 			)
 		)
+		(property "Part" "TCC0805X7R333K500DTS"
+			(at 308.61 142.24 0)
+			(hide yes)
+			(show_name no)
+			(do_not_autoplace no)
+			(effects
+				(font
+					(size 1.27 1.27)
+				)
+			)
+		)
 		(pin "1"
 		)
@@
 			)
 		)
+		(property "Part" "RCA0510KFLF"
+			(at 283.21 142.24 0)
+			(hide yes)
+			(show_name no)
+			(do_not_autoplace no)
+			(effects
+				(font
+					(size 1.27 1.27)
+				)
+			)
+		)
 		(pin "2"
 		)
@@
 			)
 		)
+		(property "Part" "0805B105M500AT"
+			(at 236.22 148.59 0)
+			(hide yes)
+			(show_name no)
+			(do_not_autoplace no)
+			(effects
+				(font
+					(size 1.27 1.27)
+				)
+			)
+		)
 		(pin "1"
 		)
@@
 			)
 		)
+		(property "Part" "SS54"
+			(at 215.9 148.59 0)
+			(hide yes)
+			(show_name no)
+			(do_not_autoplace no)
+			(effects
+				(font
+					(size 1.27 1.27)
+				)
+			)
+		)
 		(pin "2"
 		)
@@
 			(at 283.21 154.94 0)
 			(hide yes)
+			(show_name no)
+			(do_not_autoplace no)
+			(effects
+				(font
+					(size 1.27 1.27)
+				)
+			)
+		)
+		(property "Part" "SCR0805F3K3"
+			(at 283.21 154.94 0)
+			(hide yes)

Commit message: add part numbers
Parts:
- L1: Part (none) -> TMPC1265HP-470MG-D
- U1: Part (none) -> XL4015E1
Changed lines of the file:
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@@
+			)
+		)
+		(property "Part" "XL4015E1"
+			(at 198.12 135.89 0)
+			(hide yes)
+			(show_name no)
+			(do_not_autoplace no)
+			(effects
+				(font
+					(size 1.27 1.27)
+				)
 			)
 		)
@@
 			(hide yes)
 			(show_name no)
+			(do_not_autoplace no)
+			(effects
+				(font
+					(size 1.27 1.27)
+				)
+			)
+		)
+		(property "Part" "TMPC1265HP-470MG-D"
+			(at 226.06 133.35 90)
+			(hide yes)
+			(show_name no)

Commit message: lots of changes
Parts:
- C2, C3, C4: Part 0805B105M500AT -> CL21B105KBFNNNE
- C5: Part TCC0805X7R333K500DTS -> 0805B333K500NT
- R1: Part RCA0510KFLF -> 0805W8F1002T5E
- R2: Part SCR0805F3K3 -> 0805W8F3301T5E
Changed lines of the file:
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@@
 			)
 		)
-		(property "Part" "0805B105M500AT"
+		(property "Part" "CL21B105KBFNNNE"
 			(at 142.24 146.05 0)
 			(hide yes)
@@
 			)
 		)
-		(property "Part" "0805B105M500AT"
+		(property "Part" "CL21B105KBFNNNE"
 			(at 166.37 135.89 0)
 			(hide yes)
@@
 			)
 		)
-		(property "Part" "TCC0805X7R333K500DTS"
+		(property "Part" "0805B333K500NT"
 			(at 308.61 142.24 0)
 			(hide yes)
@@
 			)
 		)
-		(property "Part" "RCA0510KFLF"
+		(property "Part" "0805W8F1002T5E"
 			(at 283.21 142.24 0)
 			(hide yes)
@@
 			)
 		)
-		(property "Part" "0805B105M500AT"
+		(property "Part" "CL21B105KBFNNNE"
 			(at 236.22 148.59 0)
 			(hide yes)
@@
 			)
 		)
-		(property "Part" "SCR0805F3K3"
+		(property "Part" "0805W8F3301T5E"
 			(at 283.21 154.94 0)
 			(hide yes)
