File: power/_vref.kicad_sch (KiCad schematic)
At the start: 8 parts, among them U2 REF5050IDGK, U3 L78L06_SOT89

Commit message: lots of changes
Parts:
- C10, C7: value 1.0uF (105) 10% 25V -> 1uF (105) 10% 25V; Part 0402X105K250CT -> CL05A105KA5NQNC
- C12: footprint Capacitor_SMD:C_0805_2012Metric -> Capacitor_SMD:C_0402_1005Metric; Part FN21X104K500ECG -> CL05B104KB54PNC
- C9: Part FN21X104K500ECG -> CL05B104KB54PNC
- U2: Part REF5050AIDGKT -> REF5050AIDGKR
Changed lines of the file:
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@@
 			)
 		)
-		(property "Footprint" "Capacitor_SMD:C_0805_2012Metric"
+		(property "Footprint" "Capacitor_SMD:C_0402_1005Metric"
 			(at 89.8652 109.22 0)
 			(hide yes)
@@
 			)
 		)
-		(property "Part" "FN21X104K500ECG"
+		(property "Part" "CL05B104KB54PNC"
 			(at 88.9 105.41 0)
 			(hide yes)
@@
 			)
 		)
-		(property "Value" "1.0uF (105) 10% 25V"
+		(property "Value" "1uF (105) 10% 25V"
 			(at 194.056 120.65 90)
 			(show_name no)
@@
 			)
 		)
-		(property "Part" "0402X105K250CT"
+		(property "Part" "CL05A105KA5NQNC"
 			(at 199.39 102.87 0)
 			(hide yes)
@@
 			)
 		)
-		(property "Value" "1.0uF (105) 10% 25V"
+		(property "Value" "1uF (105) 10% 25V"
 			(at 242.316 98.552 90)
 			(show_name no)
@@
 			)
 		)
-		(property "Part" "0402X105K250CT"
+		(property "Part" "CL05A105KA5NQNC"
 			(at 247.65 90.17 0)
 			(hide yes)
@@
 			)
 		)
-		(property "Part" "FN21X104K500ECG"
+		(property "Part" "CL05B104KB54PNC"
 			(at 233.68 90.17 0)
+			(hide yes)
+			(show_name no)
+			(do_not_autoplace no)
+			(effects
+				(font
+					(size 1.27 1.27)
+				)
+			)
+		)
+		(property "Field6" ""
+			(at 233.68 90.17 90)
 			(hide yes)
 			(show_name no)
@@
 			)
 		)
-		(property "Part" "REF5050AIDGKT"
+		(property "Part" "REF5050AIDGKR"
 			(at 180.34 90.17 0)
 			(hide yes)

Commit message: use 0603 for 1uF; correct dates
Parts:
- C10, C7: value 1uF (105) 10% 25V -> 1uF (105) 10% 50V; footprint Capacitor_SMD:C_0402_1005Metric -> Capacitor_SMD:C_0603_1608Metric; Part CL05A105KA5NQNC -> CL10A105KB8NNNC
Changed lines of the file:
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@@
 	(generator_version "10.0")
 	(paper "A4")
+	(title_block
+		(date "${CURRENT_DATE}")
+	)
 	(junction
 		(at 88.9 88.9)
@@
 	(symbol
 		(lib_id "Device:C")
-		(at 199.39 102.87 0)
-		(unit 1)
-		(body_style 1)
-		(exclude_from_sim no)
-		(in_bom yes)
-		(on_board yes)
-		(in_pos_files yes)
-		(dnp no)
-		(property "Reference" "C7"
-			(at 191.262 102.87 90)
-			(show_name no)
-			(do_not_autoplace no)
-			(effects
-				(font
-					(size 1.27 1.27)
-				)
-				(justify left)
-			)
-		)
-		(property "Value" "1uF (105) 10% 25V"
-			(at 194.056 120.65 90)
-			(show_name no)
-			(do_not_autoplace no)
-			(effects
-				(font
-					(size 1.27 1.27)
-				)
-				(justify left)
-			)
-		)
-		(property "Footprint" "Capacitor_SMD:C_0402_1005Metric"
-			(at 200.3552 106.68 0)
-			(hide yes)
-			(show_name no)
-			(do_not_autoplace no)
-			(effects
-				(font
-					(size 1.27 1.27)
-				)
-			)
-		)
-		(property "Datasheet" ""
-			(at 199.39 102.87 0)
-			(hide yes)
-			(show_name no)
-			(do_not_autoplace no)
-			(effects
-				(font
-					(size 1.27 1.27)
-				)
-			)
-		)
-		(property "Description" "Unpolarized capacitor"
-			(at 199.39 102.87 0)
-			(hide yes)
-			(show_name no)
-			(do_not_autoplace no)
-			(effects
-				(font
-					(size 1.27 1.27)
-				)
-			)
-		)
-		(property "Part" "CL05A105KA5NQNC"
-			(at 199.39 102.87 0)
-			(hide yes)
-			(show_name no)
-			(do_not_autoplace no)
-			(effects
-				(font
-					(size 1.27 1.27)
-				)
-			)
-		)
-		(pin "2"
-		)
-		(pin "1"
-		)
-		(instances
-			(project "power"
-				(path "/e63e39d7-6ac0-4ffd-8aa3-1841a4541b55/98471493-5d46-4783-887d-a469b81088aa"
-					(reference "C7")
-					(unit 1)
-				)
-			)
-		)
-	)
-	(symbol
-		(lib_id "Device:C")
 		(at 247.65 90.17 0)
 		(unit 1)
@@
 			)
 		)
-		(property "Value" "1uF (105) 10% 25V"
+		(property "Value" "1uF (105) 10% 50V"
 			(at 242.316 98.552 90)
 			(show_name no)
@@
 			)
 		)
-		(property "Footprint" "Capacitor_SMD:C_0402_1005Metric"
+		(property "Footprint" "Capacitor_SMD:C_0603_1608Metric"
 			(at 248.6152 93.98 0)
 			(hide yes)
@@
 			)
 		)
-		(property "Part" "CL05A105KA5NQNC"
+		(property "Part" "CL10A105KB8NNNC"
 			(at 247.65 90.17 0)
 			(hide yes)
@@
 					(unit 1)
 				)
+			)
+		)
+	)
+	(symbol
+		(lib_id "Device:C")
+		(at 199.39 102.87 0)
+		(unit 1)
+		(body_style 1)
+		(exclude_from_sim no)
+		(in_bom yes)
+		(on_board yes)
+		(in_pos_files yes)
+		(dnp no)
+		(property "Reference" "C7"
+			(at 191.516 111.252 90)
+			(show_name no)
+			(do_not_autoplace no)
+			(effects
+				(font
+					(size 1.27 1.27)
+				)
+				(justify left)
+			)
+		)
+		(property "Value" "1uF (105) 10% 50V"
+			(at 194.056 111.252 90)
+			(show_name no)
+			(do_not_autoplace no)
+			(effects
+				(font
+					(size 1.27 1.27)
+				)
+				(justify left)
+			)
+		)
+		(property "Footprint" "Capacitor_SMD:C_0603_1608Metric"
+			(at 200.3552 106.68 0)
+			(hide yes)
+			(show_name no)
+			(do_not_autoplace no)
+			(effects
+				(font
+					(size 1.27 1.27)
+				)
+			)
+		)
+		(property "Datasheet" ""
+			(at 199.39 102.87 0)
+			(hide yes)
+			(show_name no)
+			(do_not_autoplace no)
+			(effects
+				(font
+					(size 1.27 1.27)
+				)
+			)
+		)
+		(property "Description" "Unpolarized capacitor"
+			(at 199.39 102.87 0)
+			(hide yes)
+			(show_name no)
+			(do_not_autoplace no)
+			(effects
+				(font
+					(size 1.27 1.27)
+				)
+			)
+		)
+		(property "Part" "CL10A105KB8NNNC"
+			(at 199.39 102.87 0)
+			(hide yes)
+			(show_name no)
+			(do_not_autoplace no)
+			(effects
+				(font
+					(size 1.27 1.27)
+				)
+			)
+		)
+		(pin "2"
+		)
+		(pin "1"
+		)
+		(instances
+			(project "power"
+				(path "/e63e39d7-6ac0-4ffd-8aa3-1841a4541b55/98471493-5d46-4783-887d-a469b81088aa"
+					(reference "C7")
+					(unit 1)
+				)

Commit message: change package of C16 and C20; add ChatGPT generated logo; use 220nF instead 330nF for C11
Parts:
- C11: value 330nF (334) 10% 50V -> 220nF 10% 50V; Part NL0805B334K500CPBN -> CL21B224KBFNNNE
Changed lines of the file:
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@@
 			)
 		)
-		(property "Value" "330nF (334) 10% 50V"
+		(property "Value" "220nF 10% 50V"
 			(at 48.006 123.19 90)
 			(show_name no)
@@
 			)
 		)
-		(property "Description" "Unpolarized capacitor"
+		(property "Description" "Unpolarized capacitor (was 330nF)"
 			(at 53.34 105.41 0)
 			(hide yes)
@@
 			)
 		)
-		(property "Part" "NL0805B334K500CPBN"
+		(property "Part" "CL21B224KBFNNNE"
 			(at 53.34 105.41 0)
 			(hide yes)
