File: power/_dcdc.kicad_sch (KiCad schematic)
At the start: 17 parts, among them U5 TPS56A37RPAR

Commit message: change UVLO network Better protect against reverse current outrush when disconnecting the battery with external 5V supply connected. -> VSTART=7.96V, VSTOP=7.16, hysteresis=797mV (s. https://www.ti.com/lit/ds/symlink/tps56a37.pdf?ts=1779344700851 Chapter 6.3.6)
Parts:
- R13: value 169kΩ / 1% -> 17.8kΩ / 1%; Part 0603WAF1693T5E -> PTFR0402B17K8N9
- R14: value 36.1kΩ / 1% -> 3.09kΩ / 1%; Part RT0603BRD0736K1L -> FRC0603F3091TS
Changed lines of the file:
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@@
 			)
 		)
-		(property "Value" "36.1kΩ / 1%"
+		(property "Value" "3.09kΩ / 1%"
 			(at 85.598 96.52 0)
 			(show_name no)
@@
 			)
 		)
-		(property "Part" "RT0603BRD0736K1L"
+		(property "Part" "FRC0603F3091TS"
 			(at 88.9 97.79 0)
 			(hide yes)
@@
 			)
 		)
-		(property "Value" "169kΩ / 1%"
+		(property "Value" "17.8kΩ / 1%"
 			(at 86.36 77.47 0)
 			(show_name no)
@@
 			)
 		)
-		(property "Part" "0603WAF1693T5E"
+		(property "Part" "PTFR0402B17K8N9"
 			(at 88.9 78.74 0)
 			(hide yes)

Commit message: more comments
Other:
- note added: "(under voltage lockout) to prevent reverse currents that cause brown out on the Pi when disconnecting the battery. V_start = 7.96V V_stop = 7.16V Hysteresis = 0.797V"
- note added: "Input voltage range: 24V nominal, 8V to 28V Output voltage: 5.1V Transient response, 10A load step ΔVOUT = ±5% Output ripple voltage < 50mV at CCM Output current rating 10A Operating frequency 500kHz"
- note added: "UVLO"
- note removed: "Input voltage range: 24V nominal, 5.5V to 28V Output voltage: 5V Transient response, 10A load step ΔVOUT = ±5% Output ripple voltage < 50mV at CCM Output current rating 10A Operating frequency 500kHz"
Changed lines of the file:
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@@
 		(rev "5")
 	)
-	(text "Input voltage range:	24V nominal, 5.5V to 28V\nOutput voltage:			5V\nTransient response, 10A load step ΔVOUT = ±5%\nOutput ripple voltage < 50mV at CCM\nOutput current rating 10A\nOperating frequency 500kHz"
+	(text "UVLO"
+		(exclude_from_sim no)
+		(at 85.852 49.53 0)
+		(effects
+			(font
+				(size 2.54 2.54)
+			)
+			(justify left)
+		)
+	)
+	(text "(under voltage lockout) to prevent reverse currents that cause \nbrown out on the Pi when disconnecting the battery.\nV_start    = 7.96V\nV_stop     = 7.16V\nHysteresis = 0.797V"
+		(exclude_from_sim no)
+		(at 85.598 57.404 0)
+		(effects
+			(font
+				(size 1.27 1.27)
+			)
+			(justify left)
+		)
+	)
+	(text "Input voltage range:	24V nominal, 8V to 28V\nOutput voltage:			5.1V\nTransient response, 10A load step ΔVOUT = ±5%\nOutput ripple voltage < 50mV at CCM\nOutput current rating 10A\nOperating frequency 500kHz"
 		(exclude_from_sim no)
 		(at 178.308 174.244 0)
